File: Central V2/SRP_DIN_V2/SRP_DIN_V2.kicad_sch (KiCad schematic)
At the start: 3 parts

Commit message: Changed to V2
Other:
- note added: "CHANGE BEEN ADDED IN VER2 BRANCH AND NOT IN MAIN BRANCH"
Changed lines of the file:
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@@
+		)
+	)
+	(text "CHANGE BEEN ADDED IN VER2 BRANCH AND NOT IN MAIN BRANCH"
+		(exclude_from_sim no)
+		(at 127.762 34.036 0)
+		(effects
+			(font
+				(size 2.54 2.54)
+			)
 		)
 	)
